Commit message: commit

File: src/my_robot_description/urdf/common_properties.xacro (robot description, xacro)
@@ -7,3 +7,20 @@
         <color rgba="0.5 0.5 0.5 1"/>
     </material>
+    <xacro:macro name="box_inertia" params="m x y z o_xyz o_rpy">
+        <inertial>
+            <mass value="${m}"/>
+            <origin xyz="${o_xyz}" rpy="${o_rpy}"/>
+            <inertia ixx="${(m/12)*(y*y + z*z)}" ixy="0" ixz="0"
+                iyy="${(m/12)*(x*x + z*z)}" iyz="0"
+                izz="${(m/12)*(x*x + y*y)}"/>
+        </inertial>
+    </xacro:macro>
+    <xacro:macro name="cylinder_inertia" params="m r l o_xyz o_rpy">
+        <inertial>
+            <mass value="${m}"/>
+            <origin xyz="${o_xyz}" rpy="${o_rpy}"/>
+            <inertia ixx="${(m/12)*(3*r*r + l*l)}" ixy="0" ixz="0"
+                iyy="${(m/12)*(3*r*r + l*l)}" iyz="0"
+                izz="${(m/2)*(r*r)}"/>
+    </xacro:macro>
 </robot>

File: src/my_robot_description/urdf/mobile_base.xacro (robot description, xacro)
@@ -6,21 +6,4 @@
     <xacro:property name="wheel_radius" value="0.1" />
     <xacro:property name="wheel_length" value="0.05" />
-<!--
-    <xacro:macro name="example_macro" params="a b c">
-        <link name="dummy_link">
-            <visual>
-                <geometry>
-                    <box size="${a} ${b} ${c}" />
-                </geometry>
-            </visual>
-        </link>
-    </xacro:macro>
-    <xacro:example_macro a="2" b="3" c="4"/> -->
-    <!-- <material name="blue">
-        <color rgba="0 0 0.5 1"/>
-    </material>
-    <material name="gray">
-        <color rgba="0.5 0.5 0.5 1"/>
-    </material> -->
     <link name="base_link">
         <visual>
@@ -31,4 +14,6 @@
             <material name="blue"/>
         </visual>
+        <xacro:box_inertia m="5.0" x="${base_length}" y="${base_width}" z="${base_height}"
+                            o_xyz="0 0 ${base_height/2.0}" o_rpy="0 0 0" />
     </link>
     <xacro:macro name="wheel_link" params="prefix">
@@ -45,22 +30,4 @@
     <xacro:wheel_link prefix="right" />
     <xacro:wheel_link prefix="left" />
-    <!-- <link name="right_wheel_link">
-        <visual>
-            <geometry>
-                <cylinder radius="${wheel_radius}" length="0.05"/>
-            </geometry>
-            <origin xyz="0 0 0 " rpy="${pi / 2.0} 0 0" />
-            <material name="gray" />
-        </visual>
-    </link> -->
-    <!-- <link name="left_wheel_link">
-        <visual>
-            <geometry>
-                <cylinder radius="${wheel_radius}" length="0.05"/>
-            </geometry>
-            <origin xyz="0 0 0" rpy="1.57 0 0" />
-            <material name="gray" />
-        </visual>
-    </link> -->
     <link name="caster_wheel_link">
         <visual>

Commit message: 2 commit

File: src/my_robot_description/urdf/common_properties.xacro (robot description, xacro)
@@ -23,4 +23,14 @@
                 iyy="${(m/12)*(3*r*r + l*l)}" iyz="0"
                 izz="${(m/2)*(r*r)}"/>
+            </inertial>
+    </xacro:macro>
+    <xacro:macro name="sphere_inertia" params="m r o_xyz o_rpy">
+            <inertial>
+            <mass value="${m}"/>
+            <origin xyz="${o_xyz}" rpy="${o_rpy}"/>
+            <inertia ixx="${(2/5)*m*r*r}" ixy="0" ixz="0"
+                iyy="${(2/5)*m*r*r}" iyz="0"
+                izz="${(2/5)*m*r*r}"/>
+            </inertial>
     </xacro:macro>
 </robot>

File: src/my_robot_description/urdf/mobile_base.xacro (robot description, xacro)
@@ -26,4 +26,5 @@
                 <material name="gray" />
             </visual>
+            <xacro:cylinder_inertia m="1.0" r="${wheel_radius}" l="${wheel_length}" o_xyz="0 0 0" o_rpy="${pi / 2.0} 0 0" />
         </link>
     </xacro:macro>
@@ -33,9 +34,10 @@
         <visual>
             <geometry>
-                <sphere radius="0.05"/>
+                <sphere radius="${wheel_radius / 2.0}"/>
             </geometry>
             <origin xyz="0.2 0 -0.025" rpy="1.57 0 0" />
             <material name="gray" />
         </visual>
+        <xacro:sphere_inertia m="0.5" r="${wheel_radius / 2.0}" o_xyz="0.2 0 -0.025" o_rpy="1.57 0 0" />
     </link>
     <!-- [[[joint section]]] -->
