Commit message: 3 commit

File: src/my_robot_description/urdf/mobile_base.xacro (robot description, xacro)
@@ -14,4 +14,10 @@
             <material name="blue"/>
         </visual>
+        <collision>
+            <geometry>
+                <box size="${base_length} ${base_width} ${base_height}"/>
+            </geometry>
+            <origin xyz="0 0 0.1" rpy="0 0 0"/>
+        </collision>
         <xacro:box_inertia m="5.0" x="${base_length}" y="${base_width}" z="${base_height}"
                             o_xyz="0 0 ${base_height/2.0}" o_rpy="0 0 0" />
@@ -26,4 +32,10 @@
                 <material name="gray" />
             </visual>
+            <collision>
+                <geometry>
+                    <sphere radius="${wheel_radius}" />
+                </geometry>
+                <origin xyz="0 0 0" rpy="0 0 0" />
+            </collision>
             <xacro:cylinder_inertia m="1.0" r="${wheel_radius}" l="${wheel_length}" o_xyz="0 0 0" o_rpy="${pi / 2.0} 0 0" />
         </link>
@@ -39,4 +51,10 @@
             <material name="gray" />
         </visual>
+        <collision>
+            <geometry>
+                <sphere radius="${wheel_radius / 2.0}"/>
+            </geometry>
+            <origin xyz="0.2 0 -0.025" rpy="1.57 0 0" />
+        </collision>
         <xacro:sphere_inertia m="0.5" r="${wheel_radius / 2.0}" o_xyz="0.2 0 -0.025" o_rpy="1.57 0 0" />
     </link>

Commit message: 5 commit

File: src/my_robot_description/urdf/mobile_base.xacro (robot description, xacro)
@@ -6,4 +6,5 @@
     <xacro:property name="wheel_radius" value="0.1" />
     <xacro:property name="wheel_length" value="0.05" />
+    <link name="base_footprint" />
     <link name="base_link">
         <visual>

Commit message: 6 commit

File: src/my_robot_description/urdf/mobile_base.xacro (robot description, xacro)
@@ -6,5 +6,4 @@
     <xacro:property name="wheel_radius" value="0.1" />
     <xacro:property name="wheel_length" value="0.05" />
-    <link name="base_footprint" />
     <link name="base_link">
         <visual>
